File: controlLED.kicad_pcb (KiCad board)
At the start: 2 copper layers, 2 parts, among them U1 LD1117S50TR, U2 LD1117S33TR

Commit message: ocb1
Parts:
- added C1: C, Capacitors_SMD:C_1206, F.Cu at (83.9, 1.32)
- added C2: C, Capacitors_SMD:C_1206, F.Cu at (83.8, 6.56)
- added C3: C, Capacitors_SMD:C_1206, F.Cu at (83.7, 26.9)
- added C4: C, Capacitors_SMD:C_1206, F.Cu at (83.9, 21.8)
- added C5: C, Capacitors_SMD:C_1206, F.Cu at (60.8, 20.9)
- added C6: C, Capacitors_SMD:C_1206, F.Cu at (60.8, 26.3)
- added C7: C, Capacitors_SMD:C_1206, F.Cu at (60.5, 1.85)
- added C8: C, Capacitors_SMD:C_1206, F.Cu at (60.4, 7.03)
- added CON1: BARREL_JACK, Connect:BARREL_JACK, F.Cu at (35.4, 24.0)
- added D1: LED, LEDs:LED_1206_HandSoldering, F.Cu at (144.8, 43.2)
- added J1: connector, fp:2060-452998-404, F.Cu at (213.9, 59.0)
- added J2: connector, fp:2060-452998-404, F.Cu at (213.9, 74.9)
- added J3: connector, fp:2060-452998-404, F.Cu at (213.8, 89.4)
- added J4: connector, fp:2060-452998-404, F.Cu at (214.0, 104.7)
- added J5: connector, fp:2060-452998-404, F.Cu at (78.7, 91.4)
- added J6: connector, fp:2060-452998-404, F.Cu at (78.7, 106.7)
- added J7: connector, fp:2060-452998-404, F.Cu at (78.7, 76.2)
- added J8: connector, fp:2060-452998-404, F.Cu at (78.7, 61.0)
- added J9: connector, fp:2060-452998-404, F.Cu at (92.0, 31.4)
- added P1: CONN_A0-1, fp:Grove_1x04, F.Cu at (185.4, 126.5)
- added P10: CONN_01X06, fp:Grove_1x06, F.Cu at (141.2, 127.0)
- added P11: CONN_01X02, Pin_Headers:Pin_Header_Straight_1x02_Pitch2.54mm, F.Cu at (127.0, 40.6)
- added P2: CONN_01X01, project:1Pin_12mil_VIA, F.Cu at (78.7, 27.9)
- added P3: ESP32_sparkfun, fp:connect_esp32Thing, F.Cu at (134.6, 58.4)
- added P4: CONN_01X01, project:1Pin_12mil_VIA, F.Cu at (68.2, 7.08)
- added P5: CONN_D0-1, fp:Grove_1x04, F.Cu at (157.5, 127.0)
- added P6: CONN_A0-1, fp:Grove_1x04, F.Cu at (209.7, 127.0)
- added P7: CONN_D0-1, fp:Grove_1x04, F.Cu at (174.2, 127.0)
- added P8: CONN_UART, fp:Grove_1x04, F.Cu at (98.0, 127.0)
- added P9: CONN_I2C, fp:Grove_1x04, F.Cu at (118.8, 127.0)
- added PS1: LDD-300L, fp:LDD-XXXL, F.Cu at (175.3, 55.9)
- added PS2: LDD-300L, fp:LDD-XXXL, F.Cu at (174.8, 71.0)
- added PS3: LDD-300L, fp:LDD-XXXL, F.Cu at (174.5, 86.4)
- added PS4: LDD-300L, fp:LDD-XXXL, F.Cu at (174.6, 101.6)
- added PS5: LDD-300L, fp:LDD-XXXL, F.Cu at (116.8, 94.0)
- added PS6: LDD-300L, fp:LDD-XXXL, F.Cu at (116.8, 109.2)
- added PS7: LDD-300L, fp:LDD-XXXL, F.Cu at (116.8, 78.7)
- added PS8: LDD-300L, fp:LDD-XXXL, F.Cu at (116.8, 63.5)
- added R1: 0ohm, Resistors_SMD:R_1210_HandSoldering, F.Cu at (165.1, 73.7)
- added R2: 0ohm, Resistors_SMD:R_1210_HandSoldering, F.Cu at (165.1, 81.3)
- added R3: 0ohm, Resistors_SMD:R_1210_HandSoldering, F.Cu at (165.1, 88.9)
- added R4: 0ohm, Resistors_SMD:R_1210_HandSoldering, F.Cu at (165.1, 96.5)
- added R5: 0ohm, Resistors_SMD:R_1210_HandSoldering, F.Cu at (127.0, 88.9)
- added R6: 0ohm, Resistors_SMD:R_1210_HandSoldering, F.Cu at (127.0, 96.5)
- added R7: 0ohm, Resistors_SMD:R_1210_HandSoldering, F.Cu at (127.0, 81.3)
- added R8: 0ohm, Resistors_SMD:R_1210_HandSoldering, F.Cu at (127.0, 73.7)
- added R9: 1K, Resistors_SMD:R_1210_HandSoldering, F.Cu at (135.2, 43.2)
- moved U2 99.1 mm to (73.7, 124.5)
- moved U1 63.6 mm to (114.3, 40.6), turned to 180 degrees
Connections:
- U1 pad 2: (no net) -> Net-(C3-Pad1)
- U2 pad 2: (no net) -> /VCC_1
Other:
- rule pad_to_mask_clearance: 0.2 -> 0

Commit message: pcb init
Parts:
- moved J9 76.4 mm to (168.4, 33.9)
- moved CON1 71.6 mm to (102.9, 47.9), turned to 270 degrees
- moved P6 69.2 mm to (141.2, 118.1)
- moved P7 52.9 mm to (123.9, 110.5)
- moved P10 48.1 mm to (93.6, 119.4)
- moved J6 47.0 mm to (78.7, 59.7)
- moved PS6 45.7 mm to (118.1, 63.5)
- moved P5 34.4 mm to (123.9, 119.4)
- moved R9 34.2 mm to (165.1, 59.7), turned to 0 degrees
- moved U1 32.4 mm to (142.5, 56.5), turned to 90 degrees
- moved P1 30.9 mm to (155.7, 118.1), turned to 270 degrees
- moved R6 29.2 mm to (127.0, 67.3), turned to 0 degrees
- moved P11 29.0 mm to (152.4, 54.6), turned to 90 degrees
- moved D1 23.3 mm to (165.1, 54.6)
- moved U2 21.1 mm to (85.1, 106.7), turned to 90 degrees
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Connections:
- P3 pad 11: /Din2 -> /PWM05_
- P3 pad 31: Net-(P3-Pad31) -> /Din2
- P3 pad 32: Net-(P3-Pad32) -> /Din1
- P3 pad 8: /Din1 -> /PWM06_
- R5 pad 2: Net-(P3-Pad31) -> /PWM05_
- R6 pad 2: Net-(P3-Pad32) -> /PWM06_
Other:
- board outline added: 135.9 x 74.9 mm

Commit message: fff
Parts:
- removed P2, P4: CONN_01X01, project:1Pin_12mil_VIA
- D1, R1, R2, R3, R4, R5, R6, R7, R8, R9: moved to B.Cu
- moved C7 132.2 mm to (147.3, 101.6), turned to 0 degrees
- moved C8 132.2 mm to (147.3, 106.7), turned to 0 degrees
- moved C5 120.1 mm to (134.6, 115.6), turned to 270 degrees
- moved C6 119.2 mm to (139.7, 115.6), turned to 270 degrees
- moved CON1 118.9 mm to (200.7, 115.6), turned to 90 degrees
- moved C1 94.2 mm to (149.9, 68.6), turned to 270 degrees
- moved J9 93.0 mm to (186.7, 125.1), turned to 90 degrees
- moved C2 87.2 mm to (149.9, 63.5), turned to 90 degrees
- moved C4 72.0 mm to (141.6, 64.8), turned to 180 degrees
- moved C3 71.7 mm to (141.6, 69.2), turned to 180 degrees
- moved U2 63.1 mm to (147.3, 116.8), turned to 270 degrees
- moved P6 24.9 mm to (165.1, 111.1), turned to 0 degrees
- moved PS6 23.9 mm to (118.9, 87.4)
- moved J6 22.4 mm to (80.6, 82.0)
- moved P1 20.2 mm to (174.6, 111.1), turned to 0 degrees
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Connections:
- P3 pad 31: /Din2 -> /Din1
- P3 pad 32: /Din1 -> /Din2
Routing:
- net /VCC24: track 0.00 -> 355.3 mm, vias 0 -> 2
- net GND: track 0.00 -> 215.7 mm, vias 0 -> 7
- net /VCC_1: track 0.00 -> 103.4 mm, vias 0 -> 2
- net /CS: track 0.00 -> 66.6 mm, vias 0 -> 2
- net /SCL: track 0.00 -> 60.0 mm, vias 0 -> 2
- net /SCLK: track 0.00 -> 59.7 mm, vias 0 -> 2
- net /MOSI: track 0.00 -> 59.2 mm, vias 0 -> 2
- net /Din1: track 0.00 -> 58.6 mm
- net /Din2: track 0.00 -> 57.8 mm
- net /MISO: track 0.00 -> 53.5 mm
- net Net-(P11-Pad2): track 0.00 -> 47.3 mm
- net /RX: track 0.00 -> 42.0 mm
- net /TX: track 0.00 -> 41.6 mm
- net /Ain1: track 0.00 -> 38.1 mm
- net /Ain2: track 0.00 -> 37.5 mm
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- added copper zone on B.Cu, net GND
- added copper zone on F.Cu, net GND

Commit message: version1.0
Parts:
- D1, R9: moved to F.Cu
- moved C2 2.84 mm to (147.3, 64.8), turned to 0 degrees
- moved C1 2.62 mm to (147.3, 69.2), turned to 0 degrees
- moved R1 1.36 mm to (163.8, 65.4)
- moved R9 1.36 mm to (163.7, 59.7), turned to 180 degrees
- moved PS5 1.27 mm to (119.4, 100.3)
- moved PS7 1.27 mm to (119.4, 74.9)
- moved PS8 1.27 mm to (119.4, 62.2)
- moved R2 1.27 mm to (163.8, 71.1)
- moved R3 1.27 mm to (163.8, 76.8)
- moved R4 1.27 mm to (163.8, 82.5)
- moved C3 0.63 mm to (141.0, 69.2)
- moved C4 0.63 mm to (141.0, 64.8)
- moved PS6 0.51 mm to (119.4, 87.4)
Connections:
- J1 pad 2: (no net) -> Net-(J1-Pad1)
- J1 pad 4: (no net) -> Net-(J1-Pad3)
- J2 pad 2: (no net) -> Net-(J2-Pad1)
- J2 pad 4: (no net) -> Net-(J2-Pad3)
- J3 pad 2: (no net) -> Net-(J3-Pad1)
- J3 pad 4: (no net) -> Net-(J3-Pad3)
- J4 pad 2: (no net) -> Net-(J4-Pad1)
- J4 pad 4: (no net) -> Net-(J4-Pad3)
- J5 pad 2: (no net) -> Net-(J5-Pad1)
- J5 pad 4: (no net) -> Net-(J5-Pad3)
- J6 pad 2: (no net) -> Net-(J6-Pad1)
- J6 pad 4: (no net) -> Net-(J6-Pad3)
- J7 pad 2: (no net) -> Net-(J7-Pad1)
- J7 pad 4: (no net) -> Net-(J7-Pad3)
- J8 pad 2: (no net) -> Net-(J8-Pad1)
- J8 pad 4: (no net) -> Net-(J8-Pad3)
- J9 pad 2: (no net) -> /VCC24
- J9 pad 4: (no net) -> GND
Routing:
- net /VCC24: track 355.3 -> 406.7 mm
- net GND: track 215.7 -> 249.1 mm, vias 7 -> 36
- net /SCL: track 60.0 -> 36.0 mm, vias 2 -> 0
- net Net-(C3-Pad1): track 23.0 -> 44.1 mm
- net Net-(J7-Pad1): track 7.92 -> 18.4 mm, vias 1 -> 0
- net Net-(J8-Pad1): track 9.49 -> 20.0 mm, vias 1 -> 0
- net Net-(J5-Pad3): track 9.23 -> 19.8 mm, vias 1 -> 0
- net Net-(J7-Pad3): track 9.42 -> 19.9 mm, vias 1 -> 0
- net Net-(P11-Pad2): track 47.3 -> 37.5 mm
- net Net-(J6-Pad3): track 8.76 -> 18.5 mm, vias 1 -> 0
- net Net-(J6-Pad1): track 10.1 -> 19.8 mm, vias 1 -> 0
- net Net-(J1-Pad1): track 12.2 -> 21.8 mm, vias 1 -> 0
- net Net-(J2-Pad3): track 7.92 -> 17.2 mm, vias 1 -> 0
- net Net-(J3-Pad3): track 9.42 -> 18.7 mm, vias 1 -> 0
- net Net-(J2-Pad1): track 9.42 -> 18.7 mm, vias 1 -> 0
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Other:
- board size 135.9 x 74.9 mm -> 135.9 x 75.6 mm
- board text added: "+"
- board text added: "-"
